Commit message: Fix link name and remove unnecessary links

File: zx200_description/urdf/zx200.urdf (robot description, URDF)
Before this commit: robot zx200, 14 links, 13 joints
Links:
- removed link link1
- removed link link10
- removed link link11
- removed link link12
- removed link link13
- removed link link14
- removed link link2
- removed link link3
- removed link link4
- removed link link5
- removed link link6
- removed link link7
- removed link link8
- removed link link9
- added link arm_link, mass 0.03; collision mesh filename=package://zx200_description/meshes/zx200-arm.dae; visual mesh filename=package://zx200_description/meshes/zx200-arm.dae
- added link base_link
- added link body_link, mass 0.03; collision mesh filename=package://zx200_description/meshes/zx200-body.dae; visual mesh filename=package://zx200_description/meshes/zx200-body.dae
- added link boom_link, mass 0.03; collision mesh filename=package://zx200_description/meshes/zx200-boom.dae; visual mesh filename=package://zx200_description/meshes/zx200-boom.dae
- added link bucket_link, mass 0.03; collision mesh filename=package://zx200_description/meshes/zx200-bucket.dae; visual mesh filename=package://zx200_description/meshes/zx200-bucket.dae
- added link track_link, mass 0.03; collision mesh filename=package://zx200_description/meshes/zx200-crawler.dae; visual mesh filename=package://zx200_description/meshes/zx200-crawler.dae
Joints:
- removed joint joint1
- removed joint joint10
- removed joint joint11
- removed joint joint12
- removed joint joint2
- removed joint joint3
- removed joint joint4
- removed joint joint5
- removed joint joint6
- removed joint joint7
- removed joint joint8
- removed joint joint9
- added joint arm_joint: type revolute, parent boom_link, child arm_link, origin xyz=4.7878 0.010957 2.9959, axis 0 1 0, limit lower=0.7853981633974483 upper=2.530727415391778 effort=500 velocity=6.159937255
- added joint boom_joint: type revolute, parent body_link, child boom_link, origin xyz=0.22767 -0.040187 0.83669, axis 0 1 0, limit lower=-0.3490658503988659 upper=0.9599310885968813 effort=500 velocity=6.159937255
- added joint bucket_joint: type revolute, parent arm_link, child bucket_link, origin xyz=1.8954 -0.023546 2.1809, axis 0 1 0, limit lower=-1.2217304763960306 upper=1.3962634015954636 effort=500 velocity=6.159937255
- added joint swing_joint: type continuous, parent track_link, child body_link, origin xyz=0.10787 -0.034301 1.1206, axis 0 0 1
- joint fixed: child link2 -> track_link; parent link1 -> base_link

File: zx200_description/urdf/zx200.xacro (robot description, xacro)
@@ -6,11 +6,11 @@
 	<!-- <xacro:include filename="$(find zx200_description)/urdf/materials.xacro" /> -->
 	<!-- Used for fixing robot to Gazebo 'base_link' -->
-	<link name="link1"/>
+	<link name="base_link"/>
 	<joint name="fixed" type="fixed">
-		<parent link="link1"/>
-		<child link="link2"/>
+		<parent link="base_link"/>
+		<child link="track_link"/>
 	</joint>
 	<!-- Base Link -->
-	<link name="link2">
+	<link name="track_link">
 		<visual>
 			<geometry>
@@ -32,11 +32,11 @@
 	</link>
 	<!-- body axis -->
-	<joint name="joint1" type="continuous">
+	<joint name="swing_joint" type="continuous">
 		<origin xyz="0.10787 -0.034301 1.1206"/>
 		<axis xyz="0 0 1"/>
-		<parent link="link2"/>
-		<child link="link3"/>
+		<parent link="track_link"/>
+		<child link="body_link"/>
 	</joint>
-	<link name="link3">
+	<link name="body_link">
 		<visual>
 			<origin xyz="0 0 0"/>
@@ -60,129 +60,12 @@
 	</link>
 	<!-- boom axis -->
-	<joint name="joint2" type="revolute">
+	<joint name="boom_joint" type="revolute">
 		<origin xyz="0.22767 -0.040187 0.83669"/>
 		<axis xyz="0 1 0"/>
-		<parent link="link3"/>
-		<child link="link4"/>
+		<parent link="body_link"/>
+		<child link="boom_link"/>
 		<limit lower="${radians(-20)}" upper="${radians(55)}" effort="500" velocity="6.159937255"/>
 	</joint>
-	<joint name="joint5" type="continuous">
-		<origin xyz="0.68912 -0.033576 0.23418"/>
-		<axis xyz="0 1 0"/>
-		<parent link="link3"/>
-		<child link="link7"/>
-		<mimic joint="joint2" multiplier="${61.5/70}"/>
-	</joint>
-	<gazebo>
-		<plugin name="joint5_mimic_joint_plugin"
-				filename="libroboticsgroup_upatras_gazebo_mimic_joint_plugin.so">
-			<joint>joint2</joint>
-			<mimicJoint>joint5</mimicJoint>
-			<multiplier>${60/70}</multiplier>
-			<offset>0</offset>
-			<robotNamespace>/zx200</robotNamespace>
-		</plugin>
-	</gazebo>
-	<joint name="joint6" type="prismatic">
-		<origin xyz="0 0 0"/>
-		<axis xyz="-0.2817 0 -0.74728"/>
-		<parent link="link7"/>
-		<child link="link8"/>
-		<limit lower="-2" upper="2" effort="500" velocity="6.159937255"/>
-		<mimic joint="joint2" multiplier="${0.8/1.22}"/>
-	</joint>
-	<gazebo>
-		<plugin name="joint6_mimic_joint_plugin"
-				filename="libroboticsgroup_upatras_gazebo_mimic_joint_plugin.so">
-			<joint>joint2</joint>
-			<mimicJoint>joint6</mimicJoint>
-			<multiplier>${0.39/-1.22}</multiplier>
-			<offset>0</offset>
-			<robotNamespace>/zx200</robotNamespace>
-		</plugin>
-	</gazebo>
-	<joint name="joint7" type="fixed">
-		<origin xyz="2.2875 0.017187 2.785"/>
-		<axis xyz="0 1 0"/>
-		<parent link="link4"/>
-		<child link="link9"/>
-	</joint>
-	<joint name="joint8" type="prismatic">
-		<origin xyz="0 0 0"/>
-		<axis xyz="0.48707 0 0.17284"/>
-		<parent link="link9"/>
-		<child link="link10"/>
-		<limit lower="-2" upper="2" effort="500" velocity="6.159937255"/>
-		<mimic joint="joint3" multiplier="${0.45/radians(50)}"/>
-	</joint>
-	<gazebo>
-		<plugin name="joint8_mimic_joint_plugin"
-				filename="libroboticsgroup_upatras_gazebo_mimic_joint_plugin.so">
-			<joint>joint3</joint>
-			<mimicJoint>joint8</mimicJoint>
-			<multiplier>${0.4/radians(50)}</multiplier>
-			<offset>0</offset>
-			<robotNamespace>/zx200</robotNamespace>
-		</plugin>
-	</gazebo>
-	<joint name="joint9" type="fixed">
-		<origin xyz="-0.24687 -0.007397 0.73594"/>
-		<axis xyz="0 1 0"/>
-		<parent link="link5"/>
-		<child link="link11"/>
-	</joint>
-	<joint name="joint10" type="prismatic">
-		<origin xyz="0 0 0"/>
-		<axis xyz="0.14917 0 0.16252"/>
-		<parent link="link11"/>
-		<child link="link12"/>
-		<limit lower="-2" upper="2" effort="500" velocity="6.159937255"/>
-		<mimic joint="joint4" multiplier="${-0.9/-2.79}"/>
-	</joint>
-	<gazebo>
-		<plugin name="joint10_mimic_joint_plugin"
-				filename="libroboticsgroup_upatras_gazebo_mimic_joint_plugin.so">
-			<joint>joint4</joint>
-			<mimicJoint>joint10</mimicJoint>
-			<multiplier>${-0.9/-2.79}</multiplier>
-			<offset>0</offset>
-			<robotNamespace>/zx200</robotNamespace>
-		</plugin>
-	</gazebo>
-	<joint name="joint11" type="continuous">
-		<origin xyz="1.5754 -0.01272 1.8799"/>
-		<axis xyz="0 1 0"/>
-		<parent link="link5"/>
-		<child link="link13"/>
-		<mimic joint="joint4" multiplier="${120/160}"/>
-	</joint>
-	<gazebo>
-		<plugin name="joint11_mimic_joint_plugin"
-				filename="libroboticsgroup_upatras_gazebo_mimic_joint_plugin.so">
-			<joint>joint4</joint>
-			<mimicJoint>joint11</mimicJoint>
-			<multiplier>${120/160}</multiplier>
-			<offset>0</offset>
-			<robotNamespace>/zx200</robotNamespace>
-		</plugin>
-	</gazebo>
-	<joint name="joint12" type="continuous">
-		<origin xyz="-0.32404 -0.008096 0.33854"/>
-		<axis xyz="0 1 0"/>
-		<parent link="link6"/>
-		<child link="link14"/>
-		<mimic joint="joint4" multiplier="${-210/160}"/>
-	</joint>
-	<gazebo>
-		<plugin name="joint12_mimic_joint_plugin"
-				filename="libroboticsgroup_upatras_gazebo_mimic_joint_plugin.so">
-			<joint>joint4</joint>
-			<mimicJoint>joint12</mimicJoint>
-			<multiplier>${-92/160}</multiplier>
-			<offset>0</offset>
-			<robotNamespace>/zx200</robotNamespace>
-		</plugin>
-	</gazebo>
-	<link name="link4">
+	<link name="boom_link">
 		<visual>
 			<origin xyz="0 0 0"/>
@@ -205,12 +88,12 @@
 		</inertial>
 	</link>
-	<joint name="joint3" type="revolute">
+	<joint name="arm_joint" type="revolute">
 		<origin xyz="4.7878 0.010957 2.9959"/>
 		<axis xyz="0 1 0"/>
-		<parent link="link4"/>
-		<child link="link5"/>
+		<parent link="boom_link"/>
+		<child link="arm_link"/>
 		<limit lower="${radians(45)}" upper="${radians(145)}" effort="500" velocity="6.159937255"/>
 	</joint>
-	<link name="link5">
+	<link name="arm_link">
 		<visual>
 			<origin xyz="0 0 0"/>
@@ -234,12 +117,12 @@
 	</link>
 	<!-- bucket axis -->
-	<joint name="joint4" type="revolute">
+	<joint name="bucket_joint" type="revolute">
 		<origin xyz="1.8954 -0.023546 2.1809"/>
 		<axis xyz="0 1 0"/>
-		<parent link="link5"/>
-		<child link="link6"/>
+		<parent link="arm_link"/>
+		<child link="bucket_link"/>
 		<limit lower="${radians(-70)}" upper="${radians(80)}" effort="500" velocity="6.159937255"/>
 	</joint>
-	<link name="link6">
+	<link name="bucket_link">
 		<visual>
 			<origin xyz="0 0 0"/>
@@ -262,175 +145,7 @@
 		</inertial>
 	</link>
-	<link name="link7">
-		<visual>
-			<origin xyz="0 0 0"/>
-			<geometry>
-				<mesh filename="package://zx200_description/meshes/zx200-boom-cyl1.dae"/>
-			</geometry>
-		</visual>
-		<collision>
-			<origin xyz="0 0 0"/>
-			<geometry>
-				<mesh filename="package://zx200_description/meshes/zx200-boom-cyl1.dae"/>
-			</geometry>
-		</collision>
-		<inertial>
-			<origin xyz="0 0 0" rpy="0 0 0"/>
-			<mass value="0.03"/>
-			<inertia ixx="1.0" ixy="0.0" ixz="0.0"
-								iyy="1.0" iyz="0.0"
-											izz="1.0"/>
-		</inertial>
-	</link>
-	<link name="link8">
-		<visual>
-			<origin xyz="0 0 0"/>
-			<geometry>
-				<mesh filename="package://zx200_description/meshes/zx200-boom-cyl2.dae"/>
-			</geometry>
-		</visual>
-		<collision>
-			<origin xyz="0 0 0"/>
-			<geometry>
-				<mesh filename="package://zx200_description/meshes/zx200-boom-cyl2.dae"/>
-			</geometry>
-		</collision>
-		<inertial>
-			<origin xyz="0 0 0" rpy="0 0 0"/>
-			<mass value="0.03"/>
-			<inertia ixx="1.0" ixy="0.0" ixz="0.0"
-								iyy="1.0" iyz="0.0"
-											izz="1.0"/>
-		</inertial>
-	</link>
-	<link name="link9">
-		<visual>
-			<origin xyz="0 0 0"/>
-			<geometry>
-				<mesh filename="package://zx200_description/meshes/zx200-arm-cyl1.dae"/>
-			</geometry>
-		</visual>
-		<collision>
-			<origin xyz="0 0 0"/>
-			<geometry>
-				<mesh filename="package://zx200_description/meshes/zx200-arm-cyl1.dae"/>
-			</geometry>
-		</collision>
-		<inertial>
-			<origin xyz="0 0 0" rpy="0 0 0"/>
-			<mass value="0.03"/>
-			<inertia ixx="1.0" ixy="0.0" ixz="0.0"
-								iyy="1.0" iyz="0.0"
-											izz="1.0"/>
-		</inertial>
-	</link>
-	<link name="link10">
-		<visual>
-			<origin xyz="0 0 0"/>
-			<geometry>
-				<mesh filename="package://zx200_description/meshes/zx200-arm-cyl2.dae"/>
-			</geometry>
-		</visual>
-		<collision>
-			<origin xyz="0 0 0"/>
-			<geometry>
-				<mesh filename="package://zx200_description/meshes/zx200-arm-cyl2.dae"/>
-			</geometry>
-		</collision>
-		<inertial>
-			<origin xyz="0 0 0" rpy="0 0 0"/>
-			<mass value="0.03"/>
-			<inertia ixx="1.0" ixy="0.0" ixz="0.0"
-								iyy="1.0" iyz="0.0"
-											izz="1.0"/>
-		</inertial>
-	</link>
-	<link name="link11">
-		<visual>
-			<origin xyz="0 0 0"/>
-			<geometry>
-				<mesh filename="package://zx200_description/meshes/zx200-bucket-cyl1.dae"/>
-			</geometry>
-		</visual>
-		<collision>
-			<origin xyz="0 0 0"/>
-			<geometry>
-				<mesh filename="package://zx200_description/meshes/zx200-bucket-cyl1.dae"/>
-			</geometry>
-		</collision>
-		<inertial>
-			<origin xyz="0 0 0" rpy="0 0 0"/>
-			<mass value="0.03"/>
-			<inertia ixx="1.0" ixy="0.0" ixz="0.0"
-								iyy="1.0" iyz="0.0"
-											izz="1.0"/>
-		</inertial>
-	</link>
-	<link name="link12">
-		<visual>
-			<origin xyz="0 0 0"/>
-			<geometry>
-				<mesh filename="package://zx200_description/meshes/zx200-bucket-cyl2.dae"/>
-			</geometry>
-		</visual>
-		<collision>
-			<origin xyz="0 0 0"/>
-			<geometry>
-				<mesh filename="package://zx200_description/meshes/zx200-bucket-cyl2.dae"/>
-			</geometry>
-		</collision>
-		<inertial>
-			<origin xyz="0 0 0" rpy="0 0 0"/>
-			<mass value="0.03"/>
-			<inertia ixx="1.0" ixy="0.0" ixz="0.0"
-								iyy="1.0" iyz="0.0"
-											izz="1.0"/>
-		</inertial>
-	</link>
-	<link name="link13">
-		<visual>
-			<origin xyz="0 0 0"/>
-			<geometry>
-				<mesh filename="package://zx200_description/meshes/zx200-part1.dae"/>
-			</geometry>
-		</visual>
-		<collision>
-			<origin xyz="0 0 0"/>
-			<geometry>
-				<mesh filename="package://zx200_description/meshes/zx200-part1.dae"/>
-			</geometry>
-		</collision>
-		<inertial>
-			<origin xyz="0 0 0" rpy="0 0 0"/>
-			<mass value="0.03"/>
-			<inertia ixx="1.0" ixy="0.0" ixz="0.0"
-								iyy="1.0" iyz="0.0"
-											izz="1.0"/>
-		</inertial>
-	</link>
-	<link name="link14">
-		<visual>
-			<origin xyz="0 0 0"/>
-			<geometry>
-				<mesh filename="package://zx200_description/meshes/zx200-part2.dae"/>
-			</geometry>
-		</visual>
-		<collision>
-			<origin xyz="0 0 0"/>
-			<geometry>
-				<mesh filename="package://zx200_description/meshes/zx200-part2.dae"/>
-			</geometry>
-		</collision>
-		<inertial>
-			<origin xyz="0 0 0" rpy="0 0 0"/>
-			<mass value="0.03"/>
-			<inertia ixx="1.0" ixy="0.0" ixz="0.0"
-								iyy="1.0" iyz="0.0"
-											izz="1.0"/>
-		</inertial>
-	</link>
 	<transmission name="tran1">
 		<type>transmission_interface/SimpleTransmission</type>
-		<joint name="joint1">
+		<joint name="swing_joint">
 			<hardwareInterface>hardware_interface/EffortJointInterface</hardwareInterface>
 		</joint>
@@ -442,5 +157,5 @@
 	<transmission name="tran2">
 		<type>transmission_interface/SimpleTransmission</type>
-		<joint name="joint2">
+		<joint name="boom_joint">
 			<hardwareInterface>hardware_interface/EffortJointInterface</hardwareInterface>
 		</joint>
@@ -452,5 +167,5 @@
 	<transmission name="tran3">
 		<type>transmission_interface/SimpleTransmission</type>
-		<joint name="joint3">
+		<joint name="arm_joint">
 			<hardwareInterface>hardware_interface/EffortJointInterface</hardwareInterface>
 		</joint>
@@ -462,5 +177,5 @@
 	<transmission name="tran4">
 		<type>transmission_interface/SimpleTransmission</type>
-		<joint name="joint4">
+		<joint name="bucket_joint">
 			<hardwareInterface>hardware_interface/EffortJointInterface</hardwareInterface>
 		</joint>
