Commit message: Add moveit_config pkg and ikfast_plugin pkg

File: zx200_description/urdf/zx200.xacro (robot description, xacro)
@@ -7,5 +7,5 @@
 	<!-- Used for fixing robot to Gazebo 'base_link' -->
 	<link name="base_link"/>
-	<joint name="fixed" type="fixed">
+	<joint name="base_joint" type="fixed">
 		<parent link="base_link"/>
 		<child link="track_link"/>
@@ -145,4 +145,27 @@
 		</inertial>
 	</link>
+	<link name="bucket_end_link">
+		<visual>
+			<origin xyz="0 0 0" rpy="0 0 0"/>
+			<geometry>
+				<box size="0.001 0.001 0.001" />
+			</geometry>
+			<!-- <material name="red"/> -->
+		</visual>
+		<inertial>
+			<origin xyz="0 0 0" />
+			<mass value="1.0e-03" />
+			<inertia ixx="1.0e-03" ixy="0.0" ixz="0.0"
+					iyy="1.0e-03" iyz="0.0"
+					izz="1.0e-03" />
+		</inertial>
+  	</link>
+  <joint name="bucket_end_joint" type="revolute">
+    <parent link="bucket_link"/>
+    <child link="bucket_end_link"/>
+    <axis xyz="1 0 0"/>
+    <origin rpy="0 ${radians(50)} 0" xyz="0 0 1.23"/>
+    <limit effort="1" lower="-3.14" upper="3.14" velocity="0.5"/>
+  </joint>
 	<transmission name="tran1">
 		<type>transmission_interface/SimpleTransmission</type>

File: zx200_moveit_config/config/zx200.urdf (robot description, URDF)
Before this commit: robot zx200, 6 links, 5 joints
Links:
- added link bucket_end_link, mass 1.0e-03; visual box size=0.001 0.001 0.001
Joints:
- removed joint fixed
- added joint base_joint: type fixed, parent base_link, child track_link
- added joint bucket_end_joint: type revolute, parent bucket_link, child bucket_end_link, origin xyz=0 0 1.23 rpy=0 0.8726646259971648 0, axis 1 0 0, limit lower=-3.14 upper=3.14 effort=1 velocity=0.5

Commit message: Fix to considerate with urdf on unity

File: zx200_description/urdf/zx200.xacro (robot description, xacro)
@@ -61,5 +61,5 @@
 	<!-- boom axis -->
 	<joint name="boom_joint" type="revolute">
-		<origin xyz="0.22767 -0.040187 0.83669"/>
+		<origin rpy="0 0.6108652382 0" xyz="0.22767 -0.040187 0.83669"/>
 		<axis xyz="0 1 0"/>
 		<parent link="body_link"/>
@@ -89,5 +89,5 @@
 	</link>
 	<joint name="arm_joint" type="revolute">
-		<origin xyz="4.7878 0.010957 2.9959"/>
+		<origin rpy="0 0.2617993878 0" xyz="4.7878 0.010957 2.9959"/>
 		<axis xyz="0 1 0"/>
 		<parent link="boom_link"/>
@@ -118,5 +118,5 @@
 	<!-- bucket axis -->
 	<joint name="bucket_joint" type="revolute">
-		<origin xyz="1.8954 -0.023546 2.1809"/>
+		<origin rpy="0 -0.3490658504 0" xyz="1.8954 -0.023546 2.1809"/>
 		<axis xyz="0 1 0"/>
 		<parent link="arm_link"/>
@@ -165,5 +165,5 @@
     <child link="bucket_end_link"/>
     <axis xyz="1 0 0"/>
-    <origin rpy="0 ${radians(50)} 0" xyz="0 0 1.23"/>
+    <origin rpy="0 ${radians(50)} 0" xyz="1.2 0 1"/>
     <limit effort="1" lower="-3.14" upper="3.14" velocity="0.5"/>
   </joint>

Commit message: Fix range of each joint

File: zx200_description/urdf/zx200.xacro (robot description, xacro)
@@ -61,9 +61,9 @@
 	<!-- boom axis -->
 	<joint name="boom_joint" type="revolute">
-		<origin rpy="0 0.6108652382 0" xyz="0.22767 -0.040187 0.83669"/>
+		<origin rpy="0 ${radians(35)} 0" xyz="0.22767 -0.040187 0.83669"/>
 		<axis xyz="0 1 0"/>
 		<parent link="body_link"/>
 		<child link="boom_link"/>
-		<limit lower="${radians(-20)}" upper="${radians(55)}" effort="500" velocity="6.159937255"/>
+		<limit lower="${radians(-55)}" upper="${radians(20)}" effort="500" velocity="6.159937255"/>
 	</joint>
 	<link name="boom_link">
@@ -89,9 +89,9 @@
 	</link>
 	<joint name="arm_joint" type="revolute">
-		<origin rpy="0 0.2617993878 0" xyz="4.7878 0.010957 2.9959"/>
+		<origin rpy="0 ${radians(15)} 0" xyz="4.7878 0.010957 2.9959"/>
 		<axis xyz="0 1 0"/>
 		<parent link="boom_link"/>
 		<child link="arm_link"/>
-		<limit lower="${radians(45)}" upper="${radians(145)}" effort="500" velocity="6.159937255"/>
+		<limit lower="${radians(30)}" upper="${radians(130)}" effort="500" velocity="6.159937255"/>
 	</joint>
 	<link name="arm_link">
@@ -118,9 +118,9 @@
 	<!-- bucket axis -->
 	<joint name="bucket_joint" type="revolute">
-		<origin rpy="0 -0.3490658504 0" xyz="1.8954 -0.023546 2.1809"/>
+		<origin rpy="0 ${radians(-20)} 0" xyz="1.8954 -0.023546 2.1809"/>
 		<axis xyz="0 1 0"/>
 		<parent link="arm_link"/>
 		<child link="bucket_link"/>
-		<limit lower="${radians(-70)}" upper="${radians(80)}" effort="500" velocity="6.159937255"/>
+		<limit lower="${radians(-50)}" upper="${radians(100)}" effort="500" velocity="6.159937255"/>
 	</joint>
 	<link name="bucket_link">

Commit message: Fix for IK using position of bucket joint

File: zx200_description/urdf/zx200.xacro (robot description, xacro)
@@ -165,5 +165,6 @@
     <child link="bucket_end_link"/>
     <axis xyz="1 0 0"/>
-    <origin rpy="0 ${radians(50)} 0" xyz="1.2 0 1"/>
+    <!-- <origin rpy="0 ${radians(50)} 0" xyz="1.2 0 1"/> -->
+    <origin rpy="0 0 0" xyz="0 0 0"/>
     <limit effort="1" lower="-3.14" upper="3.14" velocity="0.5"/>
   </joint>

Commit message: Fix xacro

File: zx200_description/urdf/zx200.xacro (robot description, xacro)
@@ -37,4 +37,5 @@
 		<parent link="track_link"/>
 		<child link="body_link"/>
+		<limit lower="${radians(-180)}" upper="${radians(180)}" effort="500" velocity="6.159937255"/>
 	</joint>
 	<link name="body_link">
@@ -61,5 +62,5 @@
 	<!-- boom axis -->
 	<joint name="boom_joint" type="revolute">
-		<origin rpy="0 ${radians(35)} 0" xyz="0.22767 -0.040187 0.83669"/>
+		<origin rpy="0 ${radians(32.0357)} 0" xyz="0.22767 -0.040187 0.83669"/>
 		<axis xyz="0 1 0"/>
 		<parent link="body_link"/>
@@ -89,5 +90,5 @@
 	</link>
 	<joint name="arm_joint" type="revolute">
-		<origin rpy="0 ${radians(15)} 0" xyz="4.7878 0.010957 2.9959"/>
+		<origin rpy="0 ${radians(16.9707)} 0" xyz="4.7878 0.010957 2.9959"/>
 		<axis xyz="0 1 0"/>
 		<parent link="boom_link"/>
@@ -118,9 +119,9 @@
 	<!-- bucket axis -->
 	<joint name="bucket_joint" type="revolute">
-		<origin rpy="0 ${radians(-20)} 0" xyz="1.8954 -0.023546 2.1809"/>
+		<origin rpy="0 ${radians(-9.20083)} 0" xyz="1.8954 -0.023546 2.1809"/>
 		<axis xyz="0 1 0"/>
 		<parent link="arm_link"/>
 		<child link="bucket_link"/>
-		<limit lower="${radians(-50)}" upper="${radians(100)}" effort="500" velocity="6.159937255"/>
+		<limit lower="${radians(-30)}" upper="${radians(120)}" effort="50000" velocity="6.159937255"/>
 	</joint>
 	<link name="bucket_link">
@@ -151,5 +152,4 @@
 				<box size="0.001 0.001 0.001" />
 			</geometry>
-			<!-- <material name="red"/> -->
 		</visual>
 		<inertial>
@@ -165,6 +165,5 @@
     <child link="bucket_end_link"/>
     <axis xyz="1 0 0"/>
-    <!-- <origin rpy="0 ${radians(50)} 0" xyz="1.2 0 1"/> -->
-    <origin rpy="0 0 0" xyz="0 0 0"/>
+    <origin rpy="0 0 0" xyz="1.2 0 1"/>
     <limit effort="1" lower="-3.14" upper="3.14" velocity="0.5"/>
   </joint>

Commit message: Fix to use swing_joint as continuous type

File: zx200_description/urdf/zx200.xacro (robot description, xacro)
@@ -37,5 +37,5 @@
 		<parent link="track_link"/>
 		<child link="body_link"/>
-		<limit lower="${radians(-180)}" upper="${radians(180)}" effort="500" velocity="6.159937255"/>
+		<!-- <limit lower="${radians(-360)}" upper="${radians(360)}" effort="500" velocity="6.159937255"/> -->
 	</joint>
 	<link name="body_link">

Commit message: Fix joint limit: abs(measured_value)-0.02[rad]

File: zx200_description/urdf/zx200.xacro (robot description, xacro)
@@ -37,5 +37,4 @@
 		<parent link="track_link"/>
 		<child link="body_link"/>
-		<!-- <limit lower="${radians(-360)}" upper="${radians(360)}" effort="500" velocity="6.159937255"/> -->
 	</joint>
 	<link name="body_link">
@@ -66,5 +65,5 @@
 		<parent link="body_link"/>
 		<child link="boom_link"/>
-		<limit lower="${radians(-55)}" upper="${radians(20)}" effort="500" velocity="6.159937255"/>
+		<limit lower="-1.137" upper="${radians(20)}" effort="500" velocity="6.159937255"/>
 	</joint>
 	<link name="boom_link">
@@ -94,5 +93,5 @@
 		<parent link="boom_link"/>
 		<child link="arm_link"/>
-		<limit lower="${radians(30)}" upper="${radians(130)}" effort="500" velocity="6.159937255"/>
+		<limit lower="0.594" upper="2.687" effort="500" velocity="6.159937255"/>
 	</joint>
 	<link name="arm_link">
@@ -123,5 +122,5 @@
 		<parent link="arm_link"/>
 		<child link="bucket_link"/>
-		<limit lower="${radians(-30)}" upper="${radians(120)}" effort="50000" velocity="6.159937255"/>
+		<limit lower="-0.622" upper="2.372" effort="50000" velocity="6.159937255"/>
 	</joint>
 	<link name="bucket_link">

Commit message: Fix config

File: zx200_description/urdf/zx200.xacro (robot description, xacro)
@@ -65,5 +65,5 @@
 		<parent link="body_link"/>
 		<child link="boom_link"/>
-		<limit lower="-1.137" upper="${radians(20)}" effort="500" velocity="6.159937255"/>
+		<limit lower="-1.137" upper="-0.1" effort="500" velocity="6.159937255"/>
 	</joint>
 	<link name="boom_link">

Commit message: update 251217

File: zx200_description/urdf/zx200.xacro (robot description, xacro)
@@ -65,5 +65,5 @@
 		<parent link="body_link"/>
 		<child link="boom_link"/>
-		<limit lower="-1.137" upper="-0.1" effort="500" velocity="6.159937255"/>
+		<limit lower="-1.137" upper="1.0" effort="500" velocity="6.159937255"/>
 	</joint>
 	<link name="boom_link">

Commit message: Adoption for parameters in real machine by Kyushu Universiy

File: zx200_description/urdf/zx200.xacro (robot description, xacro)
@@ -65,5 +65,5 @@
 		<parent link="body_link"/>
 		<child link="boom_link"/>
-		<limit lower="-1.137" upper="-0.1" effort="500" velocity="6.159937255"/>
+		<limit lower="-1.13" upper="1.15" effort="500" velocity="6.159937255"/>
 	</joint>
 	<link name="boom_link">
@@ -93,5 +93,5 @@
 		<parent link="boom_link"/>
 		<child link="arm_link"/>
-		<limit lower="0.594" upper="2.687" effort="500" velocity="6.159937255"/>
+		<limit lower="0.58" upper="2.687" effort="500" velocity="6.159937255"/>
 	</joint>
 	<link name="arm_link">

Commit message: update bucket_end_link joint origin parameters

File: zx200_description/urdf/zx200.xacro (robot description, xacro)
@@ -164,5 +164,5 @@
     <child link="bucket_end_link"/>
     <axis xyz="1 0 0"/>
-    <origin rpy="0 0 0" xyz="1.2 0 1"/>
+    <origin rpy="0 ${radians(105)} 0" xyz="1.25 0 0.82"/>
     <limit effort="1" lower="-3.14" upper="3.14" velocity="0.5"/>
   </joint>

Commit message: update joint rpy parameters

File: zx200_description/urdf/zx200.xacro (robot description, xacro)
@@ -118,5 +118,5 @@
 	<!-- bucket axis -->
 	<joint name="bucket_joint" type="revolute">
-		<origin rpy="0 ${radians(-9.20083)} 0" xyz="1.8954 -0.023546 2.1809"/>
+		<origin rpy="0 ${radians(-15.7415)} 0" xyz="1.8954 -0.023546 2.1809"/>
 		<axis xyz="0 1 0"/>
 		<parent link="arm_link"/>
@@ -164,5 +164,5 @@
     <child link="bucket_end_link"/>
     <axis xyz="1 0 0"/>
-    <origin rpy="0 ${radians(105)} 0" xyz="1.25 0 0.82"/>
+    <origin rpy="0 ${radians(-33.265)} 0" xyz="1.25 0 0.82"/>
     <limit effort="1" lower="-3.14" upper="3.14" velocity="0.5"/>
   </joint>
