Commit message: Modify urdf script

File: zx200_description/urdf/zx200.xacro (robot description, xacro)
@@ -61,5 +61,5 @@
 	<!-- boom axis -->
 	<joint name="boom_joint" type="revolute">
-		<origin rpy="0 ${radians(32.0357)} 0" xyz="0.22767 -0.040187 0.83669"/>
+		<origin rpy="0 ${radians(32.0357)} 0" xyz="0.05467 -0.040187 0.72492"/>
 		<axis xyz="0 1 0"/>
 		<parent link="body_link"/>
@@ -89,5 +89,5 @@
 	</link>
 	<joint name="arm_joint" type="revolute">
-		<origin rpy="0 ${radians(16.9707)} 0" xyz="4.7878 0.010957 2.9959"/>
+		<origin rpy="0 ${radians(16.9707)} 0" xyz="4.83998 0.010957 3.00227"/>
 		<axis xyz="0 1 0"/>
 		<parent link="boom_link"/>
@@ -118,5 +118,5 @@
 	<!-- bucket axis -->
 	<joint name="bucket_joint" type="revolute">
-		<origin rpy="0 ${radians(-9.20083)} 0" xyz="1.8954 -0.023546 2.1809"/>
+		<origin rpy="0 ${radians(-9.20083)} 0" xyz="1.91546 -0.023546 2.17374"/>
 		<axis xyz="0 1 0"/>
 		<parent link="arm_link"/>
@@ -164,5 +164,5 @@
     <child link="bucket_end_link"/>
     <axis xyz="1 0 0"/>
-    <origin rpy="0 0 0" xyz="1.2 0 1"/>
+    <origin rpy="0 0 0" xyz="1.13012 0 0.93856"/>
     <limit effort="1" lower="-3.14" upper="3.14" velocity="0.5"/>
   </joint>

Commit message: Fix ZX200 URDF geometry and MoveIt configuration

File: zx200_description/urdf/zx200.xacro (robot description, xacro)
@@ -61,5 +61,5 @@
 	<!-- boom axis -->
 	<joint name="boom_joint" type="revolute">
-		<origin rpy="0 ${radians(32.0357)} 0" xyz="0.22767 -0.040187 0.83669"/>
+		<origin rpy="0 ${radians(32.0357)} 0" xyz="0.05467 -0.040187 0.72492"/>
 		<axis xyz="0 1 0"/>
 		<parent link="body_link"/>
@@ -89,5 +89,5 @@
 	</link>
 	<joint name="arm_joint" type="revolute">
-		<origin rpy="0 ${radians(16.9707)} 0" xyz="4.7878 0.010957 2.9959"/>
+		<origin rpy="0 ${radians(16.9707)} 0" xyz="4.83998 0.010957 3.00227"/>
 		<axis xyz="0 1 0"/>
 		<parent link="boom_link"/>
@@ -118,5 +118,5 @@
 	<!-- bucket axis -->
 	<joint name="bucket_joint" type="revolute">
-		<origin rpy="0 ${radians(-9.20083)} 0" xyz="1.8954 -0.023546 2.1809"/>
+		<origin rpy="0 ${radians(-9.20083)} 0" xyz="1.91546 -0.023546 2.17374"/>
 		<axis xyz="0 1 0"/>
 		<parent link="arm_link"/>
@@ -152,4 +152,13 @@
 			</geometry>
 		</visual>
+		<!-- bucket_end_link is an IK tip frame, represented by the same
+		     1 mm marker for collision checking to keep the model complete
+		     without changing the bucket's practical collision envelope. -->
+		<collision>
+			<origin xyz="0 0 0" rpy="0 0 0"/>
+			<geometry>
+				<box size="0.001 0.001 0.001" />
+			</geometry>
+		</collision>
 		<inertial>
 			<origin xyz="0 0 0" />
@@ -164,5 +173,5 @@
     <child link="bucket_end_link"/>
     <axis xyz="1 0 0"/>
-    <origin rpy="0 ${radians(105)} 0" xyz="1.25 0 0.82"/>
+    <origin rpy="0 0 0" xyz="1.13012 0 0.93856"/>
     <limit effort="1" lower="-3.14" upper="3.14" velocity="0.5"/>
   </joint>

File: zx200_moveit_config/config/zx200.ros2_control.xacro (robot description, xacro)
@@ -2,5 +2,5 @@
 <robot xmlns:xacro="http://www.ros.org/wiki/xacro">
     <xacro:macro name="zx200_ros2_control" params="name plugin command_interface initial_positions_file">
-        <xacro:property name="initial_positions" value="${load_yaml(initial_positions_file)['initial_positions']}"/>
+        <xacro:property name="initial_positions" value="${xacro.load_yaml(initial_positions_file)['initial_positions']}"/>
         <ros2_control name="${name}" type="system">
             <hardware>
