Commit message: Fix to specify controller plugin in .urdf.xacro

File: zx200_moveit_config/config/zx200.ros2_control.xacro (robot description, xacro)
@@ -1,10 +1,11 @@
 <?xml version="1.0"?>
 <robot xmlns:xacro="http://www.ros.org/wiki/xacro">
-    <xacro:macro name="zx200_ros2_control" params="name initial_positions_file">
+    <xacro:macro name="zx200_ros2_control" params="name plugin initial_positions_file">
         <xacro:property name="initial_positions" value="${load_yaml(initial_positions_file)['initial_positions']}"/>
         <ros2_control name="${name}" type="system">
             <hardware>
                 <!-- By default, set up controllers for simulation. This won't work on real hardware -->
-                <plugin>mock_components/GenericSystem</plugin>
+                <!-- <plugin>mock_components/GenericSystem</plugin> -->
+                <plugin>${plugin}</plugin>
             </hardware>
             <joint name="swing_joint">

File: zx200_moveit_config/config/zx200.urdf.xacro (robot description, xacro)
@@ -6,4 +6,5 @@
     <!-- Import control_xacro -->
     <xacro:include filename="zx200.ros2_control.xacro" />
-    <xacro:zx200_ros2_control name="FakeSystem" initial_positions_file="$(arg initial_positions_file)"/>
+    <!-- <xacro:zx200_ros2_control name="FakeSystem" initial_positions_file="$(arg initial_positions_file)"/> -->
+    <xacro:zx200_ros2_control name="FakeSystem" plugin="mock_components/GenericSystem" initial_positions_file="$(arg initial_positions_file)"/>
 </robot>

Commit message: Fix to switch easily

File: zx200_moveit_config/config/zx200.ros2_control.xacro (robot description, xacro)
@@ -1,5 +1,5 @@
 <?xml version="1.0"?>
 <robot xmlns:xacro="http://www.ros.org/wiki/xacro">
-    <xacro:macro name="zx200_ros2_control" params="name plugin initial_positions_file">
+    <xacro:macro name="zx200_ros2_control" params="name plugin command_interface initial_positions_file">
         <xacro:property name="initial_positions" value="${load_yaml(initial_positions_file)['initial_positions']}"/>
         <ros2_control name="${name}" type="system">
@@ -10,7 +10,6 @@
             </hardware>
             <joint name="swing_joint">
-                <!-- <command_interface name="position"/>
-                <command_interface name="velocity"/> -->
-                <command_interface name="effort"/>
+                <!-- <command_interface name="position"/> -->
+                <command_interface name="${command_interface}"/>
                 <state_interface name="position">
                   <param name="initial_value">${initial_positions['swing_joint']}</param>
@@ -20,7 +19,6 @@
             </joint>
             <joint name="boom_joint">
-                <!-- <command_interface name="position"/>
-                <command_interface name="velocity"/> -->
-                <command_interface name="effort"/>
+                <!-- <command_interface name="position"/> -->
+                <command_interface name="${command_interface}"/>
                 <state_interface name="position">
                   <param name="initial_value">${initial_positions['boom_joint']}</param>
@@ -30,7 +28,6 @@
             </joint>
             <joint name="arm_joint">
-                <!-- <command_interface name="position"/>
-                <command_interface name="velocity"/> -->
-                <command_interface name="effort"/>
+                <!-- <command_interface name="position"/> -->
+                <command_interface name="${command_interface}"/>
                 <state_interface name="position">
                   <param name="initial_value">${initial_positions['arm_joint']}</param>
@@ -40,7 +37,6 @@
             </joint>
             <joint name="bucket_joint">
-                <!-- <command_interface name="position"/>
-                <command_interface name="velocity"/> -->
-                <command_interface name="effort"/>
+                <!-- <command_interface name="position"/> -->
+                <command_interface name="${command_interface}"/>
                 <state_interface name="position">
                   <param name="initial_value">${initial_positions['bucket_joint']}</param>
@@ -50,7 +46,6 @@
             </joint>
             <joint name="bucket_end_joint">
-                <!-- <command_interface name="position"/>
-                <command_interface name="velocity"/> -->
-                <command_interface name="effort"/>
+                <!-- <command_interface name="position"/> -->
+                <command_interface name="${command_interface}"/>
                 <state_interface name="position">
                   <param name="initial_value">${initial_positions['bucket_end_joint']}</param>
